File: COS Adapter V2.kicad_pcb (KiCad board)
At the start: 2 copper layers, 94 x 53 mm, 22 parts, among them J1 COS Input, J2 COS Output, J3 12V Input, J8 Arcom Audio, J9 Radio Audio, K1 DIP Mini Relay, Q1 2N3906, U1 LM741

Commit message: added big pads
Parts:
- C1: footprint Capacitor_THT:C_Axial_L5.1mm_D3.1mm_P7.50mm_Horizontal -> Capacitor_THT:C_Axial_L5.1mm_D3.1mm_P7.50mm_Horizontal_BIG_FEET
- R3, R4: footprint Resistor_THT:R_Axial_DIN0204_L3.6mm_D1.6mm_P7.62mm_Horizontal -> Resistor_THT:R_Axial_DIN0204_L3.6mm_D1.6mm_P7.62mm_Horizontal_BIG_FEET
Routing:
- net Net-(J8-Pin_2): track 109.0 -> 89.5 mm, vias 0 -> 1
Other:
- board text added: "Board rev 1.0"
- board text added: "Deisgn by K6KCP Board by W6DLK"
- board text added: "N/O- N/O-"
- board text removed: "Deisgn by K6KCP"
Changed lines of the file:
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@@
 		)
 	)
-	(footprint "Capacitor_THT:C_Axial_L5.1mm_D3.1mm_P7.50mm_Horizontal"
+	(footprint "Capacitor_THT:C_Axial_L5.1mm_D3.1mm_P7.50mm_Horizontal_BIG_FEET"
 		(layer "F.Cu")
 		(at 134 148.25 90)
@@
 		(tags "C Axial series Axial Horizontal pin pitch 7.5mm  length 5.1mm diameter 3.1mm")
 		(property "Reference" "C1"
-			(at -2.25 0 180)
+			(at 3.75 -2.67 90)
 			(layer "F.SilkS")
 			(effects
@@
 		(pad "1" thru_hole circle
 			(at 0 0 90)
-			(size 1.6 1.6)
-			(drill 0.8)
+			(size 2.5 2.5)
+			(drill 1)
 			(layers "*.Cu" "*.Mask")
 			(remove_unused_layers no)
@@
 		(pad "2" thru_hole circle
 			(at 7.5 0 90)
-			(size 1.6 1.6)
-			(drill 0.8)
+			(size 2.5 2.5)
+			(drill 1)
 			(layers "*.Cu" "*.Mask")
 			(remove_unused_layers no)
@@
 		)
 	)
-	(footprint "Resistor_THT:R_Axial_DIN0204_L3.6mm_D1.6mm_P7.62mm_Horizontal"
+	(footprint "Resistor_THT:R_Axial_DIN0204_L3.6mm_D1.6mm_P7.62mm_Horizontal_BIG_FEET"
 		(layer "F.Cu")
 		(at 166.5 148.31 90)
@@
 		(tags "Resistor Axial_DIN0204 series Axial Horizontal pin pitch 7.62mm 0.167W length 3.6mm diameter 1.6mm")
 		(property "Reference" "R4"
-			(at -2.19 0 180)
+			(at 3.81 -1.92 90)
 			(layer "F.SilkS")
 			(effects
@@
 		(pad "1" thru_hole circle
 			(at 0 0 90)
-			(size 1.4 1.4)
-			(drill 0.7)
+			(size 2.5 2.5)
+			(drill 1)
 			(layers "*.Cu" "*.Mask")
 			(remove_unused_layers no)
@@
 		(pad "2" thru_hole circle
 			(at 7.62 0 90)
-			(size 1.4 1.4)
-			(drill 0.7)
+			(size 2.5 2.5)
+			(drill 1)
 			(layers "*.Cu" "*.Mask")
 			(remove_unused_layers no)
@@
 		(tags "connector JST EH vertical")
 		(property "Reference" "J9"
-			(at 8.5 -3.5 180)
+			(at -3.5 -3.5 180)
 			(layer "F.SilkS")
 			(effects
@@
 		)
 	)
-	(footprint "Resistor_THT:R_Axial_DIN0204_L3.6mm_D1.6mm_P7.62mm_Horizontal"
+	(footprint "Resistor_THT:R_Axial_DIN0204_L3.6mm_D1.6mm_P7.62mm_Horizontal_BIG_FEET"
 		(layer "F.Cu")
 		(at 127.5 140.69 -90)
@@
 		(tags "Resistor Axial_DIN0204 series Axial Horizontal pin pitch 7.62mm 0.167W length 3.6mm diameter 1.6mm")
 		(property "Reference" "R3"
-			(at 9.81 0 180)
+			(at 3.81 -1.92 270)
 			(layer "F.SilkS")
 			(effects
@@
 		)
 		(property "Value" "50K"
-			(at 3.81 1.92 90)
+			(at 3.81 1.92 270)
 			(layer "F.Fab")
 			(effects
@@
 		)
 		(property "Datasheet" ""
-			(at 0 0 90)
+			(at 0 0 270)
 			(layer "F.Fab")
 			(hide yes)
@@
 		)
 		(property "Description" "Resistor"
-			(at 0 0 90)
+			(at 0 0 270)
 			(layer "F.Fab")
 			(hide yes)
@@
 		)
 		(fp_text user "${REFERENCE}"
-			(at 3.81 0 90)
+			(at 3.81 0 270)
 			(layer "F.Fab")
 			(effects
@@
 		(pad "1" thru_hole circle
 			(at 0 0 270)
-			(size 1.4 1.4)
-			(drill 0.7)
+			(size 2.5 2.5)
+			(drill 1)
 			(layers "*.Cu" "*.Mask")
 			(remove_unused_layers no)
@@
 		(pad "2" thru_hole circle
 			(at 7.62 0 270)
-			(size 1.4 1.4)
-			(drill 0.7)
+			(size 2.5 2.5)
+			(drill 1)
 			(layers "*.Cu" "*.Mask")
 			(remove_unused_layers no)
@@
 		(tags "connector JST EH vertical")
 		(property "Reference" "J2"
-			(at 7 0 180)
+			(at 6.5 0 180)
 			(layer "F.SilkS")
 			(effects
@@
 		(tags "connector JST EH vertical")
 		(property "Reference" "J8"
-			(at 8.5 -3 0)
+			(at 9 0.3 0)
 			(layer "F.SilkS")
 			(effects
@@
 	)
 	(gr_text "+"
-		(at 114.5 126.5 0)
+		(at 114 126 0)
 		(layer "F.SilkS")
 		(effects
@@
 		)
 	)
-	(gr_text "+"
-		(at 109.4 129.85 0)
+	(gr_text "12V"
+		(at 103 123 270)
 		(layer "F.SilkS")
 		(effects
 			(font
-				(size 1 1)
-				(thickness 0.1)
+				(size 2 2)
+				(thickness 0.2)
 			)
 			(justify left bottom)
 		)
 	)
-	(gr_text "12V"
-		(at 103 123 270)
+	(gr_text "N/O-\nN/O-"
+		(at 179.29 122.5 0)
 		(layer "F.SilkS")
 		(effects
 			(font
-				(size 2 2)
+				(size 1.6 1.5)
 				(thickness 0.2)
+				(bold yes)
 			)
-			(justify left bottom)
+			(justify right bottom)
 		)
 	)
@@
 		)
 	)
+	(gr_text "Board rev 1.0"
+		(at 173.5 151 0)
+		(layer "F.SilkS")
+		(effects
+			(font
+				(size 1 0.8)
+				(thickness 0.1)
+			)
+			(justify left bottom)
+		)
+	)
 	(gr_text "Radio\nAudio"
 		(at 105 139 270)
@@
 	)
 	(gr_text "RCA"
-		(at 117.5 131.5 0)
+		(at 112.5 128.5 0)
 		(layer "F.SilkS")
 		(effects
@@
 		)
 	)
-	(gr_text "Deisgn by K6KCP"
-		(at 171.5 110 0)
+	(gr_text "Deisgn by K6KCP\nBoard by W6DLK"
+		(at 182 111 0)
 		(layer "F.SilkS")
 		(effects
@@
 				(thickness 0.1)
 			)
-			(justify left bottom)
+			(justify right bottom)
 		)
 	)
@@
 	)
 	(segment
-		(start 134 142.5)
-		(end 144.59 142.5)
+		(start 161.5 141.5)
+		(end 161.5 144.41)
 		(width 0.3)
-		(layer "B.Cu")
+		(layer "F.Cu")
 		(net 16)
 	)
-	(segment
-		(start 144.59 142.5)
-		(end 146.5 144.41)
-		(width 0.3)
-		(layer "B.Cu")
+	(via
+		(at 161.5 141.5)
+		(size 0.6)
+		(drill 0.3)
+		(layers "F.Cu" "B.Cu")
 		(net 16)
 	)
 	(segment
-		(start 182 144.5)
-		(end 181.91 144.41)
+		(start 134 140.75)
+		(end 142.84 140.75)
 		(width 0.3)
 		(layer "B.Cu")
@@
 	)
 	(segment
-		(start 178 134.5)
-		(end 170 142.5)
+		(start 131.25 143.5)
+		(end 131 143.5)
 		(width 0.3)
 		(layer "B.Cu")
@@
 	)
 	(segment
-		(start 126 142.5)
-		(end 134 142.5)
+		(start 134 140.75)
+		(end 131.25 143.5)
 		(width 0.3)
 		(layer "B.Cu")
@@
 	)
 	(segment
-		(start 114 139)
-		(end 122.5 139)
+		(start 144.59 142.5)
+		(end 146.5 144.41)
 		(width 0.3)
 		(layer "B.Cu")
@@
 	)
 	(segment
-		(start 149.41 141.5)
-		(end 163.5 141.5)
+		(start 182 144.5)
+		(end 181.91 144.41)
 		(width 0.3)
 		(layer "B.Cu")
@@
 	)
 	(segment
-		(start 183.5 143)
-		(end 182 144.5)
+		(start 114 139)
+		(end 121.5 139)
 		(width 0.3)
 		(layer "B.Cu")
@@
 	)
 	(segment
-		(start 164.5 142.5)
-		(end 170 142.5)
+		(start 149.41 141.5)
+		(end 161.5 141.5)
 		(width 0.3)
 		(layer "B.Cu")
@@
 	)
 	(segment
-		(start 180.7 134.5)
-		(end 178 134.5)
+		(start 183.5 143)
+		(end 182 144.5)
 		(width 0.3)
 		(layer "B.Cu")
@@
 	)
 	(segment
-		(start 180.7 134.5)
-		(end 182.5 134.5)
+		(start 142.84 140.75)
+		(end 144.59 142.5)
 		(width 0.3)
 		(layer "B.Cu")
@@
 	)
 	(segment
-		(start 134 140.75)
-		(end 134 142.5)
+		(start 180.7 134.5)
+		(end 182.5 134.5)
 		(width 0.3)
 		(layer "B.Cu")
@@
 	)
 	(segment
-		(start 122.5 139)
-		(end 126 142.5)
+		(start 121.5 139)
+		(end 126 143.5)
 		(width 0.3)
 		(layer "B.Cu")
@@
 	)
 	(segment
-		(start 163.5 141.5)
-		(end 164.5 142.5)
+		(start 126 143.5)
+		(end 131 143.5)
 		(width 0.3)
 		(layer "B.Cu")
@@
 	)
 	(segment
-		(start 123.31 136.5)
-		(end 127.5 140.69)
+		(start 114 136.5)
+		(end 121.5 136.5)
 		(width 0.3)
 		(layer "B.Cu")
@@
 	)
 	(segment
-		(start 114 136.5)
-		(end 123.31 136.5)
+		(start 121.5 136.5)
+		(end 125.69 140.69)
+		(width 0.3)
+		(layer "B.Cu")
+		(net 20)
+	)
+	(segment
+		(start 125.69 140.69)
+		(end 127.5 140.69)
 		(width 0.3)
 		(layer "B.Cu")

Commit message: add Arcom mounting holes
Parts:
- removed H (x4): MountingHole_3.2mm_M3, MountingHole:MountingHole_3.2mm_M3
- added H1: MountingHole_3.2mm_M3_DIN965_Pad, MountingHole:MountingHole_3.2mm_M3_DIN965_Pad, F.Cu at (103.5, 103.0)
- added H2: MountingHole_3.2mm_M3_DIN965_Pad, MountingHole:MountingHole_3.2mm_M3_DIN965_Pad, F.Cu at (103.5, 112.5)
- added H3: MountingHole_3.2mm_M3_DIN965_Pad, MountingHole:MountingHole_3.2mm_M3_DIN965_Pad, F.Cu at (103.5, 150.0)
- added H4: MountingHole_3.2mm_M3_DIN965_Pad, MountingHole:MountingHole_3.2mm_M3_DIN965_Pad, F.Cu at (190.5, 103.0)
- added H5: MountingHole_3.2mm_M3_DIN965_Pad, MountingHole:MountingHole_3.2mm_M3_DIN965_Pad, F.Cu at (183.5, 112.5)
- added H6: MountingHole_3.2mm_M3_DIN965_Pad, MountingHole:MountingHole_3.2mm_M3_DIN965_Pad, F.Cu at (183.5, 150.0)
- added H7: MountingHole_3.2mm_M3_DIN965_Pad, MountingHole:MountingHole_3.2mm_M3_DIN965_Pad, F.Cu at (190.5, 150.0)
- moved J2 1.78 mm to (180.7, 123.2)

Commit message: fill in the foil
Routing:
- added copper zone on B.Cu, net (none)
- added copper zone on B.Cu, net GND
Other:
- board text added: "Board rev 1.1"
- board text removed: "Board rev 1.0"
Changed lines of the file:
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@@
 			(outputformat 1)
 			(mirror no)
-			(drillshape 1)
+			(drillshape 0)
 			(scaleselection 1)
-			(outputdirectory "")
+			(outputdirectory "Fabrication/")
 		)
 	)
@@
 		)
 	)
-	(gr_text "Board rev 1.0"
+	(gr_text "Board rev 1.1"
 		(at 170.5 151 0)
 		(layer "F.SilkS")
@@
 		(net 21)
 	)
+	(zone
+		(net 1)
+		(net_name "GND")
+		(layer "B.Cu")
+		(hatch edge 0.5)
+		(connect_pads
+			(clearance 0.8)
+		)
+		(min_thickness 0.25)
+		(filled_areas_thickness no)
+		(fill yes
+			(thermal_gap 0.5)
+			(thermal_bridge_width 0.5)
+		)
+		(polygon
+			(pts
+				(xy 195.5 98) (xy 96 98) (xy 96 156) (xy 196 155.5) (xy 197.5 151.5)
+			)
+		)
+	)
+	(zone
+		(net 0)
+		(net_name "")
+		(layer "B.Cu")
+		(hatch edge 0.5)
+		(priority 1)
+		(connect_pads
+			(clearance 0.5)
+		)
+		(min_thickness 0.25)
+		(filled_areas_thickness no)
+		(fill yes
+			(thermal_gap 0.5)
+			(thermal_bridge_width 0.5)
+			(island_removal_mode 1)
+			(island_area_min 10)
+		)
+		(polygon
+			(pts
+				(xy 179 133) (xy 175.5 133) (xy 169 139.5) (xy 169 142.5) (xy 173.5 142.5) (xy 179 137)
+			)
+		)
+	)
 	(embedded_fonts no)

Commit message: v2.2: fix diode polarity
Parts:
- moved D2 7.62 mm to (155.2, 118.7), turned to -90 degrees
Connections:
- D2 pad 1: GND -> Net-(D2-K)
- D2 pad 2: Net-(D2-A) -> GND
- K1 pad 2: Net-(D2-A) -> Net-(D2-K)
- Q1 pad 1: Net-(D2-A) -> Net-(D2-K)
- R2 pad 2: Net-(D2-A) -> Net-(D2-K)
Routing:
- net Net-(D2-K): track 0.00 -> 23.9 mm
- net Net-(D2-A): track 23.9 -> 0.00 mm
Other:
- board text added: "Board rev 2.2"
- board text removed: "Board rev 1.1"
Changed lines of the file:
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@@
 	(net 9 "unconnected-(U1-NULL-Pad1)")
 	(net 10 "unconnected-(U1-NC-Pad8)")
-	(net 11 "Net-(D2-A)")
+	(net 11 "Net-(D2-K)")
 	(net 12 "Net-(J1-Pin_1)")
 	(net 13 "Net-(J2-Pin_2)")
@@
 			(layers "*.Cu" "*.Mask")
 			(remove_unused_layers no)
-			(net 11 "Net-(D2-A)")
+			(net 11 "Net-(D2-K)")
 			(pintype "passive")
 		)
@@
 			(layers "*.Cu" "*.Mask")
 			(remove_unused_layers no)
-			(net 11 "Net-(D2-A)")
+			(net 11 "Net-(D2-K)")
 			(pinfunction "E")
 			(pintype "passive")
@@
 	(footprint "Diode_THT:D_A-405_P7.62mm_Horizontal"
 		(layer "F.Cu")
-		(at 155.25 126.31 90)
+		(at 155.25 118.69 -90)
 		(descr "Diode, A-405 series, Axial, Horizontal, pin pitch=7.62mm, length*diameter=5.2*2.7mm^2, http://www.diodes.com/_files/packages/A-405.pdf")
 		(tags "Diode A-405 series Axial Horizontal pin pitch 7.62mm  length 5.2mm diameter 2.7mm")
@@
 		)
 		(property "Sim.Device" "D"
-			(at 0 0 90)
+			(at 0 0 270)
 			(unlocked yes)
 			(layer "F.Fab")
@@
 		)
 		(property "Sim.Pins" "1=K 2=A"
-			(at 0 0 90)
+			(at 0 0 270)
 			(unlocked yes)
 			(layer "F.Fab")
@@
 		(attr through_hole)
 		(fp_line
-			(start 6.53 -1.47)
-			(end 6.53 -1.14)
+			(start 1.09 1.47)
+			(end 6.53 1.47)
 			(stroke
 				(width 0.12)
@@
 		)
 		(fp_line
-			(start 2.11 -1.47)
-			(end 2.11 1.47)
+			(start 6.53 1.47)
+			(end 6.53 1.14)
 			(stroke
 				(width 0.12)
@@
 		)
 		(fp_line
-			(start 1.99 -1.47)
-			(end 1.99 1.47)
+			(start 1.09 1.14)
+			(end 1.09 1.47)
 			(stroke
 				(width 0.12)
@@
 		)
 		(fp_line
-			(start 1.87 -1.47)
-			(end 1.87 1.47)
+			(start 1.09 -1.14)
+			(end 1.09 -1.47)
 			(stroke
 				(width 0.12)
@@
 		)
 		(fp_line
-			(start 1.09 -1.14)
-			(end 1.09 -1.47)
+			(start 1.87 -1.47)
+			(end 1.87 1.47)
 			(stroke
 				(width 0.12)
@@
 		)
 		(fp_line
-			(start 1.09 1.14)
-			(end 1.09 1.47)
+			(start 1.99 -1.47)
+			(end 1.99 1.47)
 			(stroke
 				(width 0.12)
@@
 		)
 		(fp_line
-			(start 6.53 1.47)
-			(end 6.53 1.14)
+			(start 2.11 -1.47)
+			(end 2.11 1.47)
 			(stroke
 				(width 0.12)
@@
 		)
 		(fp_line
-			(start 1.09 1.47)
-			(end 6.53 1.47)
+			(start 6.53 -1.47)
+			(end 6.53 -1.14)
 			(stroke
 				(width 0.12)
@@
 		)
 		(fp_line
-			(start 2.09 -1.35)
-			(end 2.09 1.35)
+			(start 0 0)
+			(end 1.21 0)
 			(stroke
 				(width 0.1)
@@
 		)
 		(fp_line
-			(start 1.99 -1.35)
-			(end 1.99 1.35)
+			(start 7.62 0)
+			(end 6.41 0)
 			(stroke
 				(width 0.1)
@@
 		)
 		(fp_line
-			(start 7.62 0)
-			(end 6.41 0)
+			(start 1.99 -1.35)
+			(end 1.99 1.35)
 			(stroke
 				(width 0.1)
@@
 		)
 		(fp_line
-			(start 0 0)
-			(end 1.21 0)
+			(start 2.09 -1.35)
+			(end 2.09 1.35)
 			(stroke
 				(width 0.1)
@@
 		)
 		(pad "1" thru_hole roundrect
-			(at 0 0 90)
+			(at 0 0 270)
 			(size 1.8 1.8)
 			(drill 0.9)
@@
 			(remove_unused_layers no)
 			(roundrect_rratio 0.138889)
-			(net 1 "GND")
+			(net 11 "Net-(D2-K)")
 			(pinfunction "K")
 			(pintype "passive")
 		)
 		(pad "2" thru_hole circle
-			(at 7.62 0 90)
+			(at 7.62 0 270)
 			(size 1.8 1.8)
 			(drill 0.9)
 			(layers "*.Cu" "*.Mask")
 			(remove_unused_layers no)
-			(net 11 "Net-(D2-A)")
+			(net 1 "GND")
 			(pinfunction "A")
 			(pintype "passive")
@@
 			(layers "*.Cu" "*.Mask")
 			(remove_unused_layers no)
-			(net 11 "Net-(D2-A)")
+			(net 11 "Net-(D2-K)")
 			(pintype "passive")
 		)
@@
 		)
 	)
-	(gr_text "Board rev 1.1"
+	(gr_text "Board rev 2.2"
 		(at 170.5 151 0)
 		(layer "F.SilkS")
